File: KiCad/main_pcb/_restore_backup_2026-07-21T15-07-55-405/main_pcb.kicad_sch (KiCad schematic)
At the start: 5 parts

Commit message: Starts work on Main PCB
Connections:
- net D/C: no longer U5.22 (GPA1)
- net MOSI: no longer U5.24 (GPA3)
- net RST_EYES: no longer U5.21 (GPA0)
- net SCK: no longer U5.23 (GPA2)
- net VCC: no longer U1.10 (V_{SS}), U1.9 (V_{DD}), U2.7 (VCC), U3.7 (VCC), U5.10 (V_{SS}), U5.9 (V_{DD})
- net CS_EYE_R: no longer names the net of U5.25 (GPA4)
- net EYE_LEFT.CS_EYE_L: no longer names the net of U2.2 (CS)
- net EYE_LEFT.CS_EYE_L: no longer U1.5 (GPB4)
- net EYE_LEFT.D/C: no longer names the net of U2.3 (DC)
- net EYE_LEFT.D/C: no longer U1.2 (GPB1)
- net EYE_LEFT.MOSI: no longer names the net of U2.4 (MOSI)
- net EYE_LEFT.MOSI: no longer U1.4 (GPB3)
- net EYE_LEFT.RST_EYES: no longer names the net of U2.1 (RST)
- net EYE_LEFT.RST_EYES: no longer U1.1 (GPB0)
- net EYE_LEFT.SCK: no longer names the net of U2.5 (CLK)
- net EYE_LEFT.SCK: no longer U1.3 (GPB2)
- net EYE_RIGHT.CS_EYE_R: no longer names the net of U5.5 (GPB4)
- net EYE_RIGHT.CS_EYE_R: no longer U3.2 (CS)
- net EYE_RIGHT.D/C: no longer names the net of U5.2 (GPB1)
- net EYE_RIGHT.D/C: no longer U3.3 (DC)
- net EYE_RIGHT.MOSI: no longer names the net of U5.4 (GPB3)
- net EYE_RIGHT.MOSI: no longer U3.4 (MOSI)
- net EYE_RIGHT.RST_EYES: no longer names the net of U5.1 (GPB0)
- net EYE_RIGHT.RST_EYES: no longer U3.1 (RST)
- net EYE_RIGHT.SCK: no longer names the net of U5.3 (GPB2)
- net EYE_RIGHT.SCK: no longer U3.5 (CLK)
- new net 3V3: U1.10 (V_{SS}), U5.10 (V_{SS})
- new net 5V: U1.9 (V_{DD}), U5.9 (V_{DD})
- no-connect marks 28 -> 0
Other:
- moved on the sheet: U4
