File: KiCad/main_pcb/USB-C.kicad_sch (KiCad schematic)
At the start: 9 parts, among them J2 USB-C, U10 JSMSEMI AMS1117-3.3V, U8 CH340C

Commit message: feat(KiCad): Continues work on circuit
Parts:
- J2: symbol Lily's_Pad:USB_TYPE-C-31-M-14 -> lilys_pad:USB_TYPE-C-31-M-14
- U10: symbol Lily's_Pad:JSMSEMI_AMS1117-3.3V -> lilys_pad:JSMSEMI_AMS1117-3.3V
- U8: symbol Lily's_Pad:CH340C -> lilys_pad:CH340C
Other:
- moved on the sheet: U10
Changed lines of the file:
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@@
+	)
+	(junction
+		(at 168.91 95.25)
+		(diameter 0)
+		(color 0 0 0 0)
 	)
 	(junction
@@
 		(color 0 0 0 0)
 	)
+	(junction
+		(at 67.31 115.57)
+		(diameter 0)
+		(color 0 0 0 0)
+	)
 	(no_connect
 		(at 68.58 97.79)
@@
 	(wire
 		(pts
+			(xy 168.91 95.25) (xy 168.91 97.79)
+		)
+		(stroke
+			(width 0)
+			(type default)
+		)
+	)
+	(wire
+		(pts
 			(xy 57.15 115.57) (xy 59.69 115.57)
 		)
@@
 	(wire
 		(pts
-			(xy 168.91 86.36) (xy 168.91 97.79)
+			(xy 168.91 86.36) (xy 168.91 95.25)
 		)
 		(stroke
@@
 	(wire
 		(pts
+			(xy 153.67 76.2) (xy 153.67 78.74)
+		)
+		(stroke
+			(width 0)
+			(type default)
+		)
+	)
+	(wire
+		(pts
+			(xy 67.31 115.57) (xy 68.58 115.57)
+		)
+		(stroke
+			(width 0)
+			(type default)
+		)
+	)
+	(wire
+		(pts
 			(xy 88.9 105.41) (xy 138.43 105.41)
 		)
@@
 	(wire
 		(pts
-			(xy 66.04 115.57) (xy 68.58 115.57)
+			(xy 66.04 115.57) (xy 67.31 115.57)
 		)
 		(stroke
@@
 	)
 	(symbol
-		(lib_id "Lily's_Pad:USB_TYPE-C-31-M-14")
+		(lib_id "lilys_pad:USB_TYPE-C-31-M-14")
 		(at 168.91 106.68 0)
 		(unit 1)
@@
 	)
 	(symbol
-		(lib_id "Lily's_Pad:CH340C")
+		(lib_id "lilys_pad:CH340C")
 		(at 78.74 106.68 180)
 		(unit 1)
@@
 		(fields_autoplaced yes)
 		(property "Reference" "U8"
-			(at 78.74 123.19 0)
+			(at 78.74 90.17 0)
 			(show_name no)
 			(do_not_autoplace no)
@@
 		)
 		(property "Value" "CH340C"
-			(at 78.74 120.65 0)
+			(at 78.74 92.71 0)
 			(show_name no)
 			(do_not_autoplace no)
@@
 	)
 	(symbol
-		(lib_id "Lily's_Pad:JSMSEMI_AMS1117-3.3V")
-		(at 144.78 73.66 180)
+		(lib_id "lilys_pad:PWR_FLG")
+		(at 166.37 95.25 270)
+		(unit 1)
+		(body_style 1)
+		(exclude_from_sim no)
+		(in_bom no)
+		(on_board no)
+		(in_pos_files yes)
+		(dnp no)
+		(fields_autoplaced yes)
+		(property "Reference" "#PWR042"
+			(at 166.37 95.25 0)
+			(hide yes)
+			(show_name no)
+			(do_not_autoplace no)
+			(effects
+				(font
+					(size 1.27 1.27)
+				)
+			)
+		)
+		(property "Value" "PWR_FLG"
+			(at 166.37 95.25 0)
+			(hide yes)
+			(show_name no)
+			(do_not_autoplace no)
+			(effects
+				(font
+					(size 1.27 1.27)
+				)
+			)
+		)
+		(property "Footprint" ""
+			(at 166.37 95.25 0)
+			(hide yes)
+			(show_name no)
+			(do_not_autoplace no)
+			(effects
+				(font
+					(size 1.27 1.27)
+				)
+			)
+		)
+		(property "Datasheet" ""
+			(at 166.37 95.25 0)
+			(hide yes)
+			(show_name no)
+			(do_not_autoplace no)
+			(effects
+				(font
+					(size 1.27 1.27)
+				)
+			)
+		)
+		(property "Description" ""
+			(at 166.37 95.25 0)
+			(hide yes)
+			(show_name no)
+			(do_not_autoplace no)
+			(effects
+				(font
+					(size 1.27 1.27)
+				)
+			)
+		)
+		(pin "1"
+		)
+		(instances
+			(project "main_pcb"
+				(path "/346fb29b-2426-4b69-9f9a-e979b6e41832/a4816677-4d4e-4f2e-882a-ab61f6eb2b02"
+					(reference "#PWR042")
+					(unit 1)
+				)
+			)
+		)
+	)
+	(symbol
+		(lib_id "lilys_pad:JSMSEMI_AMS1117-3.3V")
+		(at 144.78 73.66 0)
 		(unit 1)
 		(body_style 1)
@@
 		(dnp no)
 		(property "Reference" "U10"
-			(at 137.16 74.9301 90)
+			(at 143.256 87.63 0)
 			(show_name no)
 			(do_not_autoplace no)
@@
 		)
 		(property "Value" "JSMSEMI AMS1117-3.3V"
-			(at 144.526 61.976 90)
+			(at 145.034 85.344 90)
 			(show_name no)
 			(do_not_autoplace no)
@@
 	(symbol
 		(lib_id "lilys_pad:GND")
-		(at 156.21 76.2 90)
+		(at 153.67 81.28 0)
 		(unit 1)
 		(body_style 1)
@@
 		(dnp no)
 		(property "Reference" "#PWR022"
-			(at 158.75 76.2 0)
+			(at 153.67 83.82 0)
 			(hide yes)
 			(show_name no)
@@
 		)
 		(property "Value" "GND"
-			(at 158.496 76.2 0)
+			(at 153.67 83.566 0)
 			(show_name no)
 			(do_not_autoplace no)
@@
 		)
 		(property "Footprint" ""
-			(at 156.21 76.2 0)
+			(at 153.67 81.28 0)
 			(hide yes)
 			(show_name no)
@@
 		)
 		(property "Datasheet" ""
-			(at 156.21 76.2 0)
+			(at 153.67 81.28 0)
 			(hide yes)
 			(show_name no)
@@
 		)
 		(property "Description" ""
-			(at 156.21 76.2 0)
+			(at 153.67 81.28 0)
 			(hide yes)
 			(show_name no)
@@
 		(in_pos_files yes)
 		(dnp no)
-		(fields_autoplaced yes)
 		(property "Reference" "#PWR023"
 			(at 143.51 102.87 0)
@@
 		)
 		(property "Value" "GND"
-			(at 145.415 99.06 90)
+			(at 143.764 102.616 0)
 			(show_name no)
 			(do_not_autoplace no)
@@
 					(unit 1)
 				)
+			)
+		)
+	)
+	(symbol
+		(lib_id "lilys_pad:PWR_FLG")
+		(at 67.31 118.11 0)
+		(unit 1)
+		(body_style 1)
+		(exclude_from_sim no)
+		(in_bom no)
+		(on_board no)
+		(in_pos_files yes)
+		(dnp no)
+		(fields_autoplaced yes)
+		(property "Reference" "#PWR041"
+			(at 67.31 118.11 0)
+			(hide yes)
+			(show_name no)
+			(do_not_autoplace no)
+			(effects
+				(font
+					(size 1.27 1.27)
+				)
+			)
+		)
+		(property "Value" "PWR_FLG"
+			(at 67.31 118.11 0)
+			(hide yes)
+			(show_name no)
+			(do_not_autoplace no)
+			(effects
+				(font
+					(size 1.27 1.27)
+				)
+			)
+		)
+		(property "Footprint" ""
+			(at 67.31 118.11 0)
+			(hide yes)
+			(show_name no)
+			(do_not_autoplace no)
+			(effects
+				(font
+					(size 1.27 1.27)
+				)
+			)
+		)
+		(property "Datasheet" ""
+			(at 67.31 118.11 0)
+			(hide yes)
+			(show_name no)
+			(do_not_autoplace no)
+			(effects
+				(font
+					(size 1.27 1.27)
+				)
+			)
+		)
+		(property "Description" ""
+			(at 67.31 118.11 0)
+			(hide yes)
+			(show_name no)
+			(do_not_autoplace no)
+			(effects
+				(font
+					(size 1.27 1.27)
+				)
+			)
+		)
+		(pin "1"
+		)
+		(instances
+			(project "main_pcb"
+				(path "/346fb29b-2426-4b69-9f9a-e979b6e41832/a4816677-4d4e-4f2e-882a-ab61f6eb2b02"
+					(reference "#PWR041")
+					(unit 1)
+				)

Commit message: feat(KiCad): Continues work on circuit
Parts:
- R2, R3: value 5.1k -> 5.1kΩ
Changed lines of the file:
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@@
 		(in_pos_files yes)
 		(dnp no)
-		(fields_autoplaced yes)
 		(property "Reference" "R3"
-			(at 184.15 104.14 90)
-			(show_name no)
-			(do_not_autoplace no)
-			(effects
-				(font
-					(size 1.27 1.27)
-				)
-			)
-		)
-		(property "Value" "5.1k"
-			(at 184.15 106.68 90)
+			(at 184.15 112.776 90)
+			(show_name no)
+			(do_not_autoplace no)
+			(effects
+				(font
+					(size 1.27 1.27)
+				)
+			)
+		)
+		(property "Value" "5.1kΩ"
+			(at 184.15 115.316 90)
 			(show_name no)
 			(do_not_autoplace no)
@@
 		(in_pos_files yes)
 		(dnp no)
-		(fields_autoplaced yes)
 		(property "Reference" "R2"
-			(at 153.67 96.52 90)
-			(show_name no)
-			(do_not_autoplace no)
-			(effects
-				(font
-					(size 1.27 1.27)
-				)
-			)
-		)
-		(property "Value" "5.1k"
-			(at 153.67 99.06 90)
-			(show_name no)
-			(do_not_autoplace no)
+			(at 153.67 97.79 90)
+			(show_name no)
+			(do_not_autoplace no)
+			(effects
+				(font
+					(size 1.27 1.27)
+				)
+			)
+		)
+		(property "Value" "5.1kΩ"
+			(at 153.67 100.33 90)
+			(show_name no)
+			(do_not_autoplace no)
