File: KiCad/main_pcb/usb-c.kicad_sch (KiCad schematic)
At the start: 16 parts, among them J5 Conn_01x02, J6 USB_C_Receptacle_USB2.0_14P, U5 AMS1117-3.3, U7 CH340C

Commit message: feat(3D models): Adds 3D models to PCB
Parts:
- U5: footprint Package_TO_SOT_SMD:SOT-223-3_TabPin2 -> Lilibrary:SOT-223-3_TabPin2_AMS1117
Changed lines of the file:
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@@
 			)
 		)
-		(property "Footprint" "Package_TO_SOT_SMD:SOT-223-3_TabPin2"
+		(property "Footprint" "Lilibrary:SOT-223-3_TabPin2_AMS1117"
 			(at 198.12 67.31 0)
 			(effects

Commit message: feat(pcb): Uses new footprint for Male Header 2x13
Parts:
- U5: footprint Lilibrary:SOT-223-3_TabPin2_AMS1117 -> Package_TO_SOT_SMD:SOT-223-3_TabPin2
Changed lines of the file:
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@@
 			)
 		)
-		(property "Footprint" "Lilibrary:SOT-223-3_TabPin2_AMS1117"
+		(property "Footprint" "Package_TO_SOT_SMD:SOT-223-3_TabPin2"
 			(at 198.12 67.31 0)
 			(effects
