File: KiCad/main_pcb/usb-c.kicad_sch (KiCad schematic)
At the start: 16 parts, among them J2 Conn_01x02, J6 USB_C_Receptacle_USB2.0_14P, U5 CH340C, U6 AMS1117-3.3

Commit message: chore(migration): Migrates to homebrew symbols for PCB.
Parts:
- C19: renamed from C16; LCSC C19702 -> C14663
- J6: footprint Connector_USB:USB_C_Receptacle_HRO_TYPE-C-31-M-12 -> Lilibrary:USB-C (Home-brew); symbol Connector:USB_C_Receptacle_USB2.0_14P -> Lilybrary:USB-C
- R8: renamed from R9; value 10kΩ -> 330Ω
- U5: renamed from U6; footprint Package_TO_SOT_SMD:SOT-223-3_TabPin2 -> Lilibrary:SOT-223-3_TabPin2_AMS1117
- U7: renamed from U5; footprint Package_SO:SOIC-16_3.9x9.9mm_P1.27mm -> Lilibrary:SOP-16_CH340C
- renumbered C20 to C15, C18 to C16, C14 to C17, C15 to C18, C17 to C20, C19 to C21, C21 to C7, J2 to J5, R8 to R7, R7 to R9
Connections:
- net GND: now also J6.S2 (SHIELD), J6.S3 (SHIELD), J6.S4 (SHIELD)
Changed lines of the file:
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@@
 	)
 	(junction
-		(at 106.68 134.62)
+		(at 114.3 124.46)
 		(diameter 0)
 		(color 0 0 0 0)
@@
 	(wire
 		(pts
-			(xy 106.68 134.62) (xy 106.68 135.89)
+			(xy 114.3 124.46) (xy 114.3 125.73)
 		)
 		(stroke
@@
 	(wire
 		(pts
+			(xy 113.03 124.46) (xy 113.03 121.92)
+		)
+		(stroke
+			(width 0)
+			(type default)
+		)
+	)
+	(wire
+		(pts
 			(xy 160.02 63.5) (xy 160.02 72.39)
 		)
@@
 	(wire
 		(pts
+			(xy 115.57 124.46) (xy 115.57 121.92)
+		)
+		(stroke
+			(width 0)
+			(type default)
+		)
+	)
+	(wire
+		(pts
+			(xy 113.03 124.46) (xy 114.3 124.46)
+		)
+		(stroke
+			(width 0)
+			(type default)
+		)
+	)
+	(wire
+		(pts
 			(xy 140.97 125.73) (xy 148.59 125.73)
 		)
@@
 	(wire
 		(pts
-			(xy 102.87 134.62) (xy 106.68 134.62)
-		)
-		(stroke
-			(width 0)
-			(type default)
-		)
-	)
-	(wire
-		(pts
-			(xy 106.68 134.62) (xy 110.49 134.62)
+			(xy 114.3 124.46) (xy 115.57 124.46)
 		)
 		(stroke
@@
 		(on_board yes)
 		(dnp no)
-		(property "Reference" "C19"
+		(property "Reference" "C21"
 			(at 171.45 127.508 90)
 			(effects
@@
 			(project "main_pcb"
 				(path "/ecf3cf27-e370-4cc5-86a4-628206277f58/0e6b288a-4b38-488e-b038-c06265dff781"
-					(reference "C19")
+					(reference "C21")
 					(unit 1)
 				)
@@
 		(dnp no)
 		(fields_autoplaced yes)
-		(property "Reference" "C21"
+		(property "Reference" "C7"
 			(at 214.63 67.3099 0)
 			(effects
@@
 			(project "main_pcb"
 				(path "/ecf3cf27-e370-4cc5-86a4-628206277f58/0e6b288a-4b38-488e-b038-c06265dff781"
-					(reference "C21")
+					(reference "C7")
 					(unit 1)
 				)
@@
 		(on_board yes)
 		(dnp no)
-		(property "Reference" "C15"
+		(property "Reference" "C18"
 			(at 150.876 58.42 0)
 			(effects
@@
 			(project "main_pcb"
 				(path "/ecf3cf27-e370-4cc5-86a4-628206277f58/0e6b288a-4b38-488e-b038-c06265dff781"
-					(reference "C15")
+					(reference "C18")
 					(unit 1)
 				)
@@
 		(on_board yes)
 		(dnp no)
-		(property "Reference" "U6"
+		(property "Reference" "U5"
 			(at 193.04 69.342 0)
 			(effects
@@
 			)
 		)
-		(property "Footprint" "Package_TO_SOT_SMD:SOT-223-3_TabPin2"
+		(property "Footprint" "Lilibrary:SOT-223-3_TabPin2_AMS1117"
 			(at 198.12 67.31 0)
 			(effects
@@
 			(project "main_pcb"
 				(path "/ecf3cf27-e370-4cc5-86a4-628206277f58/0e6b288a-4b38-488e-b038-c06265dff781"
-					(reference "U6")
+					(reference "U5")
 					(unit 1)
 				)
@@
 		(on_board yes)
 		(dnp no)
-		(property "Reference" "U5"
+		(property "Reference" "U7"
 			(at 160.8933 140.97 0)
 			(effects
@@
 			)
 		)
-		(property "Footprint" "Package_SO:SOIC-16_3.9x9.9mm_P1.27mm"
+		(property "Footprint" "Lilibrary:SOP-16_CH340C"
 			(at 140.208 95.504 0)
 			(effects
@@
 			(project "main_pcb"
 				(path "/ecf3cf27-e370-4cc5-86a4-628206277f58/0e6b288a-4b38-488e-b038-c06265dff781"
-					(reference "U5")
+					(reference "U7")
 					(unit 1)
 				)
@@
 		(on_board yes)
 		(dnp no)
-		(property "Reference" "C18"
+		(property "Reference" "C16"
 			(at 162.56 103.378 90)
 			(effects
@@
 			(project "main_pcb"
 				(path "/ecf3cf27-e370-4cc5-86a4-628206277f58/0e6b288a-4b38-488e-b038-c06265dff781"
-					(reference "C18")
+					(reference "C16")
 					(unit 1)
 				)
@@
 	)
 	(symbol
-		(lib_id "Connector:USB_C_Receptacle_USB2.0_14P")
-		(at 110.49 111.76 0)
+		(lib_id "Lilybrary:USB-C")
+		(at 116.84 106.68 0)
 		(unit 1)
 		(exclude_from_sim no)
@@
 		(fields_autoplaced yes)
 		(property "Reference" "J6"
-			(at 110.49 88.9 0)
+			(at 116.84 88.9 0)
 			(effects
 				(font
@@
 		)
 		(property "Value" "USB_C_Receptacle_USB2.0_14P"
-			(at 110.49 91.44 0)
-			(effects
-				(font
-					(size 1.27 1.27)
-				)
-			)
-		)
-		(property "Footprint" "Connector_USB:USB_C_Receptacle_HRO_TYPE-C-31-M-12"
-			(at 114.3 111.76 0)
+			(at 116.84 91.44 0)
+			(effects
+				(font
+					(size 1.27 1.27)
+				)
+			)
+		)
+		(property "Footprint" "Lilibrary:USB-C (Home-brew)"
+			(at 116.84 106.68 0)
 			(effects
 				(font
@@
 		)
 		(property "Datasheet" "https://www.usb.org/sites/default/files/documents/usb_type-c.zip"
-			(at 114.3 111.76 0)
+			(at 116.84 106.68 0)
 			(effects
 				(font
@@
 		)
 		(property "Description" "USB 2.0-only 14P Type-C Receptacle connector"
-			(at 110.49 111.76 0)
+			(at 116.84 106.68 0)
 			(effects
 				(font
@@
 		)
 		(property "KLC_S3.3" ""
-			(at 110.49 111.76 0)
+			(at 116.84 106.68 0)
 			(effects
 				(font
@@
 		)
 		(property "KLC_S4.1" ""
-			(at 110.49 111.76 0)
+			(at 116.84 106.68 0)
 			(effects
 				(font
@@
 		)
 		(property "LCSC" "C165948"
-			(at 110.49 111.76 0)
+			(at 116.84 106.68 0)
 			(effects
 				(font
@@
 		)
 		(pin "A7"
+		)
+		(pin "S2"
+		)
+		(pin "S3"
+		)
+		(pin "S4"
 		)
 		(instances
@@
 		(on_board yes)
 		(dnp no)
-		(property "Reference" "C17"
+		(property "Reference" "C20"
 			(at 162.56 93.218 90)
 			(effects
@@
 			(project "main_pcb"
 				(path "/ecf3cf27-e370-4cc5-86a4-628206277f58/0e6b288a-4b38-488e-b038-c06265dff781"
-					(reference "C17")
+					(reference "C20")
 					(unit 1)
 				)
@@
 		(on_board yes)
 		(dnp no)
-		(property "Reference" "R9"
+		(property "Reference" "R8"
 			(at 124.46 64.77 90)
 			(effects
@@
 			)
 		)
-		(property "Value" "10kΩ"
+		(property "Value" "330Ω"
 			(at 126.746 61.976 90)
 			(effects
@@
 			(project "main_pcb"
 				(path "/ecf3cf27-e370-4cc5-86a4-628206277f58/0e6b288a-4b38-488e-b038-c06265dff781"
-					(reference "R9")
+					(reference "R8")
 					(unit 1)
 				)
@@
 	(symbol
 		(lib_id "power:GND")
-		(at 106.68 135.89 0)
+		(at 114.3 125.73 0)
 		(unit 1)
 		(exclude_from_sim no)
@@
 		(fields_autoplaced yes)
 		(property "Reference" "#PWR036"
-			(at 106.68 142.24 0)
+			(at 114.3 132.08 0)
 			(effects
 				(font
@@
 		)
 		(property "Value" "GND"
-			(at 106.68 140.97 0)
+			(at 114.3 130.81 0)
 			(effects
 				(font
@@
 		)
 		(property "Footprint" ""
-			(at 106.68 135.89 0)
+			(at 114.3 125.73 0)
 			(effects
 				(font
@@
 		)
 		(property "Datasheet" ""
-			(at 106.68 135.89 0)
+			(at 114.3 125.73 0)
 			(effects
 				(font
@@
 		)
 		(property "Description" "Power symbol creates a global label with name \"GND\" , ground"
-			(at 106.68 135.89 0)
+			(at 114.3 125.73 0)
 			(effects
 				(font
@@
 		(on_board yes)
 		(dnp no)
-		(property "Reference" "C20"
+		(property "Reference" "C15"
 			(at 182.88 67.3099 0)
 			(effects
@@
 			(project "main_pcb"
 				(path "/ecf3cf27-e370-4cc5-86a4-628206277f58/0e6b288a-4b38-488e-b038-c06265dff781"
-					(reference "C20")
+					(reference "C15")
 					(unit 1)
 				)
@@
 		(on_board yes)
 		(dnp no)
-		(property "Reference" "R8"
+		(property "Reference" "R7"
 			(at 129.54 104.14 90)
 			(effects
@@
 			(project "main_pcb"
 				(path "/ecf3cf27-e370-4cc5-86a4-628206277f58/0e6b288a-4b38-488e-b038-c06265dff781"
-					(reference "R8")
+					(reference "R7")
 					(unit 1)
 				)
@@
 		(on_board yes)
 		(dnp no)
-		(property "Reference" "C14"
+		(property "Reference" "C17"
 			(at 139.446 58.42 0)
 			(effects
@@
 			(project "main_pcb"
 				(path "/ecf3cf27-e370-4cc5-86a4-628206277f58/0e6b288a-4b38-488e-b038-c06265dff781"
-					(reference "C14")
+					(reference "C17")
 					(unit 1)
 				)
@@
 		(on_board yes)
 		(dnp no)
-		(property "Reference" "C16"
+		(property "Reference" "C19"
 			(at 162.306 58.42 0)
 			(effects
@@
 			)
 		)
-		(property "LCSC" "C19702"
+		(property "LCSC" "C14663"
 			(at 160.02 59.69 0)
 			(effects
@@
 			(project "main_pcb"
 				(path "/ecf3cf27-e370-4cc5-86a4-628206277f58/0e6b288a-4b38-488e-b038-c06265dff781"
-					(reference "C16")
+					(reference "C19")
 					(unit 1)
 				)
@@
 		(dnp no)
 		(fields_autoplaced yes)
-		(property "Reference" "J2"
+		(property "Reference" "J5"
 			(at 138.43 93.9799 0)
 			(effects
@@
 			(project "main_pcb"
 				(path "/ecf3cf27-e370-4cc5-86a4-628206277f58/0e6b288a-4b38-488e-b038-c06265dff781"
-					(reference "J2")
+					(reference "J5")
 					(unit 1)
 				)
@@
 		(on_board yes)
 		(dnp no)
-		(property "Reference" "R7"
+		(property "Reference" "R9"
 			(at 129.54 101.6 90)
 			(effects
@@
 			(project "main_pcb"
 				(path "/ecf3cf27-e370-4cc5-86a4-628206277f58/0e6b288a-4b38-488e-b038-c06265dff781"
-					(reference "R7")
+					(reference "R9")
 					(unit 1)
 				)

Commit message: feat(pcb): I think that's about right
Parts:
- C15, C16, C17, C18, C19, C20, C21, C7: footprint Capacitor_SMD:C_0603_1608Metric_Pad1.08x0.95mm_HandSolder -> Lilibrary:Capacitor_0603
- D5: footprint LED_SMD:LED_0603_1608Metric_Pad1.05x0.95mm_HandSolder -> Lilibrary:LED_0603
- J6: footprint Lilibrary:USB-C (Home-brew) -> Lilibrary:USB_C_Receptacle_HRO_TYPE-C-31-M-12
- R7, R8, R9: footprint Resistor_SMD:R_0603_1608Metric_Pad0.98x0.95mm_HandSolder -> Lilibrary:Resistor_0603
Changed lines of the file:
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@@
 			)
 		)
-		(property "Footprint" "Capacitor_SMD:C_0603_1608Metric_Pad1.08x0.95mm_HandSolder"
+		(property "Footprint" "Lilibrary:Capacitor_0603"
 			(at 176.53 132.3848 0)
 			(effects
@@
 			)
 		)
-		(property "Footprint" "Capacitor_SMD:C_0603_1608Metric_Pad1.08x0.95mm_HandSolder"
+		(property "Footprint" "Lilibrary:Capacitor_0603"
 			(at 211.7852 72.39 0)
 			(effects
@@
 			)
 		)
-		(property "Footprint" "Capacitor_SMD:C_0603_1608Metric_Pad1.08x0.95mm_HandSolder"
+		(property "Footprint" "Lilibrary:Capacitor_0603"
 			(at 149.5552 63.5 0)
 			(effects
@@
 			)
 		)
-		(property "Footprint" "LED_SMD:LED_0603_1608Metric_Pad1.05x0.95mm_HandSolder"
+		(property "Footprint" "Lilibrary:LED_0603"
 			(at 124.46 54.61 0)
 			(effects
@@
 			)
 		)
-		(property "Footprint" "Capacitor_SMD:C_0603_1608Metric_Pad1.08x0.95mm_HandSolder"
+		(property "Footprint" "Lilibrary:Capacitor_0603"
 			(at 167.64 108.2548 0)
 			(effects
@@
 			)
 		)
-		(property "Footprint" "Lilibrary:USB-C (Home-brew)"
+		(property "Footprint" "Lilibrary:USB_C_Receptacle_HRO_TYPE-C-31-M-12"
 			(at 116.84 106.68 0)
 			(effects
@@
 			)
 		)
-		(property "Footprint" "Capacitor_SMD:C_0603_1608Metric_Pad1.08x0.95mm_HandSolder"
+		(property "Footprint" "Lilibrary:Capacitor_0603"
 			(at 167.64 98.0948 0)
 			(effects
@@
 			)
 		)
-		(property "Footprint" "Resistor_SMD:R_0603_1608Metric_Pad0.98x0.95mm_HandSolder"
+		(property "Footprint" "Lilibrary:Resistor_0603"
 			(at 126.238 64.77 90)
 			(effects
@@
 			)
 		)
-		(property "Footprint" "Capacitor_SMD:C_0603_1608Metric_Pad1.08x0.95mm_HandSolder"
+		(property "Footprint" "Lilibrary:Capacitor_0603"
 			(at 180.0352 72.39 0)
 			(effects
@@
 			)
 		)
-		(property "Footprint" "Resistor_SMD:R_0603_1608Metric_Pad0.98x0.95mm_HandSolder"
+		(property "Footprint" "Lilibrary:Resistor_0603"
 			(at 129.54 105.918 90)
 			(effects
@@
 			)
 		)
-		(property "Footprint" "Capacitor_SMD:C_0603_1608Metric_Pad1.08x0.95mm_HandSolder"
+		(property "Footprint" "Lilibrary:Capacitor_0603"
 			(at 138.1252 63.5 0)
 			(effects
@@
 			)
 		)
-		(property "Footprint" "Capacitor_SMD:C_0603_1608Metric_Pad1.08x0.95mm_HandSolder"
+		(property "Footprint" "Lilibrary:Capacitor_0603"
 			(at 160.9852 63.5 0)
 			(effects
@@
 			)
 		)
-		(property "Footprint" "Resistor_SMD:R_0603_1608Metric_Pad0.98x0.95mm_HandSolder"
+		(property "Footprint" "Lilibrary:Resistor_0603"
 			(at 129.54 103.378 90)
 			(effects

Commit message: feat(schematic): Changes LED's resistor values from 330 ohms to 1k ohms.
Parts:
- R8: value 330Ω -> 1kΩ; LCSC C2933198 -> C22548
Changed lines of the file:
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@@
 			)
 		)
-		(property "Value" "330Ω"
+		(property "Value" "1kΩ"
 			(at 126.746 61.976 90)
 			(effects
@@
 			)
 		)
-		(property "LCSC" "C2933198"
+		(property "LCSC" "C22548"
 			(at 124.46 64.77 90)
 			(effects

Commit message: feat(pcb): Adds all the remaning 3D models
Parts:
- J5: footprint Connector_JST:JST_XH_B2B-XH-A_1x02_P2.50mm_Vertical -> Lilibrary:JST XH 2 pins
Connections:
- net GND: no longer J6.S2 (SHIELD), J6.S3 (SHIELD), J6.S4 (SHIELD)
- no-connect marks 6 -> 8
Changed lines of the file:
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@@
+	)
+	(no_connect
+		(at 107.95 97.79)
 	)
 	(no_connect
@@
 	(no_connect
 		(at 168.91 130.81)
+	)
+	(no_connect
+		(at 107.95 100.33)
 	)
 	(wire
@@
 		(pin "A7"
 		)
-		(pin "S2"
-		)
-		(pin "S3"
-		)
-		(pin "S4"
+		(pin "B8"
+		)
+		(pin "A8"
 		)
 		(instances
@@
 			)
 		)
-		(property "Footprint" "Connector_JST:JST_XH_B2B-XH-A_1x02_P2.50mm_Vertical"
+		(property "Footprint" "Lilibrary:JST XH 2 pins"
 			(at 135.89 93.98 0)
 			(effects

Commit message: chore: Adds 3D models to footprint, instead of adding manually when placing components :3
Parts:
- U5: footprint Lilibrary:SOT-223-3_TabPin2_AMS1117 -> Package_TO_SOT_SMD:SOT-223-3_TabPin2
- U7: footprint Lilibrary:SOP-16_CH340C -> Package_SO:SOIC-16_3.9x9.9mm_P1.27mm
Changed lines of the file:
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@@
 			)
 		)
-		(property "Footprint" "Lilibrary:SOT-223-3_TabPin2_AMS1117"
+		(property "Footprint" "Package_TO_SOT_SMD:SOT-223-3_TabPin2"
 			(at 198.12 67.31 0)
 			(effects
@@
 			)
 		)
-		(property "Footprint" "Lilibrary:SOP-16_CH340C"
+		(property "Footprint" "Package_SO:SOIC-16_3.9x9.9mm_P1.27mm"
 			(at 140.208 95.504 0)
 			(effects
@@
 			)
 		)
-		(property "Description" "USB 2.0-only 14P Type-C Receptacle connector"
+		(property "Description" ""
 			(at 116.84 106.68 0)
 			(effects

Commit message: chore
Parts:
- C19: LCSC C14663 -> C1691
- renumbered C7 to C10, C15 to C12, C21 to C16, C20 to C17, C17 to C20, C16 to C21, D5 to D4, J5 to J6, J6 to J7, R8 to R6, R7 to R8, U5 to U4, U7 to U6
Changed lines of the file:
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@@
 		(on_board yes)
 		(dnp no)
-		(property "Reference" "C21"
+		(property "Reference" "C16"
 			(at 171.45 127.508 90)
 			(effects
@@
 			)
 		)
-		(property "Description" "Unpolarized capacitor"
+		(property "Description" ""
 			(at 172.72 133.35 0)
 			(effects
@@
 			(project "main_pcb"
 				(path "/ecf3cf27-e370-4cc5-86a4-628206277f58/0e6b288a-4b38-488e-b038-c06265dff781"
-					(reference "C21")
+					(reference "C16")
 					(unit 1)
 				)
@@
 		(dnp no)
 		(fields_autoplaced yes)
-		(property "Reference" "C7"
+		(property "Reference" "C10"
 			(at 214.63 67.3099 0)
 			(effects
@@
 			)
 		)
-		(property "Description" "Unpolarized capacitor"
+		(property "Description" ""
 			(at 210.82 68.58 0)
 			(effects
@@
 			(project "main_pcb"
 				(path "/ecf3cf27-e370-4cc5-86a4-628206277f58/0e6b288a-4b38-488e-b038-c06265dff781"
-					(reference "C7")
+					(reference "C10")
 					(unit 1)
 				)
@@
 			)
 		)
-		(property "Description" "Unpolarized capacitor"
+		(property "Description" ""
 			(at 148.59 59.69 0)
 			(effects
@@
 		(dnp no)
 		(fields_autoplaced yes)
-		(property "Reference" "D5"
+		(property "Reference" "D4"
 			(at 127 51.7524 90)
 			(effects
@@
 			)
 		)
-		(property "Description" "Light emitting diode"
+		(property "Description" ""
 			(at 124.46 54.61 0)
 			(effects
@@
 			(project "main_pcb"
 				(path "/ecf3cf27-e370-4cc5-86a4-628206277f58/0e6b288a-4b38-488e-b038-c06265dff781"
-					(reference "D5")
+					(reference "D4")
 					(unit 1)
 				)
@@
 		(on_board yes)
 		(dnp no)
-		(property "Reference" "U5"
+		(property "Reference" "U4"
 			(at 193.04 69.342 0)
 			(effects
@@
 			)
 		)
-		(property "Description" "1A Low Dropout regulator, positive, 3.3V fixed output, SOT-223"
+		(property "Description" ""
 			(at 198.12 72.39 0)
 			(effects
@@
 			(project "main_pcb"
 				(path "/ecf3cf27-e370-4cc5-86a4-628206277f58/0e6b288a-4b38-488e-b038-c06265dff781"
-					(reference "U5")
+					(reference "U4")
 					(unit 1)
 				)
@@
 		(on_board yes)
 		(dnp no)
-		(property "Reference" "U7"
+		(property "Reference" "U6"
 			(at 160.8933 140.97 0)
 			(effects
@@
 			)
 		)
-		(property "Description" "USB serial converter, crystal-less, UART, SOIC-16"
+		(property "Description" ""
 			(at 157.226 89.662 0)
 			(effects
@@
 			(project "main_pcb"
 				(path "/ecf3cf27-e370-4cc5-86a4-628206277f58/0e6b288a-4b38-488e-b038-c06265dff781"
-					(reference "U7")
+					(reference "U6")
 					(unit 1)
 				)
@@
 		(on_board yes)
 		(dnp no)
-		(property "Reference" "C16"
+		(property "Reference" "C21"
 			(at 162.56 103.378 90)
 			(effects
@@
 			)
 		)
-		(property "Description" "Unpolarized capacitor"
+		(property "Description" ""
 			(at 163.83 109.22 0)
 			(effects
@@
 			(project "main_pcb"
 				(path "/ecf3cf27-e370-4cc5-86a4-628206277f58/0e6b288a-4b38-488e-b038-c06265dff781"
-					(reference "C16")
+					(reference "C21")
 					(unit 1)
 				)
@@
 		(dnp no)
 		(fields_autoplaced yes)
-		(property "Reference" "J6"
+		(property "Reference" "J7"
 			(at 116.84 88.9 0)
 			(effects
@@
 			(project "main_pcb"
 				(path "/ecf3cf27-e370-4cc5-86a4-628206277f58/0e6b288a-4b38-488e-b038-c06265dff781"
-					(reference "J6")
+					(reference "J7")
 					(unit 1)
 				)
@@
 		(on_board yes)
 		(dnp no)
-		(property "Reference" "C20"
+		(property "Reference" "C17"
 			(at 162.56 93.218 90)
 			(effects
@@
 			)
 		)
-		(property "Description" "Unpolarized capacitor"
+		(property "Description" ""
 			(at 163.83 99.06 0)
 			(effects
@@
 			(project "main_pcb"
 				(path "/ecf3cf27-e370-4cc5-86a4-628206277f58/0e6b288a-4b38-488e-b038-c06265dff781"
-					(reference "C20")
+					(reference "C17")
 					(unit 1)
 				)
@@
 		(on_board yes)
 		(dnp no)
-		(property "Reference" "R8"
+		(property "Reference" "R6"
 			(at 124.46 64.77 90)
 			(effects
@@
 			)
 		)
-		(property "Description" "Resistor"
+		(property "Description" ""
 			(at 124.46 64.77 0)
 			(effects
@@
 			(project "main_pcb"
 				(path "/ecf3cf27-e370-4cc5-86a4-628206277f58/0e6b288a-4b38-488e-b038-c06265dff781"
-					(reference "R8")
+					(reference "R6")
 					(unit 1)
 				)
@@
 		(on_board yes)
 		(dnp no)
-		(property "Reference" "C15"
+		(property "Reference" "C12"
 			(at 182.88 67.3099 0)
 			(effects
@@
 			)
 		)
-		(property "Description" "Unpolarized capacitor"
+		(property "Description" ""
 			(at 179.07 68.58 0)
 			(effects
@@
 			(project "main_pcb"
 				(path "/ecf3cf27-e370-4cc5-86a4-628206277f58/0e6b288a-4b38-488e-b038-c06265dff781"
-					(reference "C15")
+					(reference "C12")
 					(unit 1)
 				)
@@
 		(on_board yes)
 		(dnp no)
-		(property "Reference" "R7"
+		(property "Reference" "R8"
 			(at 129.54 104.14 90)
 			(effects
@@
 			)
 		)
-		(property "Description" "Resistor"
+		(property "Description" ""
 			(at 129.54 104.14 0)
 			(effects
@@
 			(project "main_pcb"
 				(path "/ecf3cf27-e370-4cc5-86a4-628206277f58/0e6b288a-4b38-488e-b038-c06265dff781"
-					(reference "R7")
+					(reference "R8")
 					(unit 1)
 				)
@@
 		(on_board yes)
 		(dnp no)
-		(property "Reference" "C17"
+		(property "Reference" "C20"
 			(at 139.446 58.42 0)
 			(effects
@@
 			)
 		)
-		(property "Description" "Unpolarized capacitor"
+		(property "Description" ""
 			(at 137.16 59.69 0)
 			(effects
@@
 			(project "main_pcb"
 				(path "/ecf3cf27-e370-4cc5-86a4-628206277f58/0e6b288a-4b38-488e-b038-c06265dff781"
-					(reference "C17")
+					(reference "C20")
 					(unit 1)
 				)
@@
 			)
 		)
-		(property "Description" "Unpolarized capacitor"
+		(property "Description" ""
 			(at 160.02 59.69 0)
 			(effects
@@
 			)
 		)
-		(property "LCSC" "C14663"
+		(property "LCSC" "C1691"
 			(at 160.02 59.69 0)
 			(effects
@@
 		(dnp no)
 		(fields_autoplaced yes)
-		(property "Reference" "J5"
+		(property "Reference" "J6"
 			(at 138.43 93.9799 0)
 			(effects
@@
 			)
 		)
-		(property "Description" "Generic connector, single row, 01x02, script generated (kicad-library-utils/schlib/autogen/connector/)"
+		(property "Description" ""
 			(at 135.89 93.98 0)
 			(effects
@@
 			(project "main_pcb"
 				(path "/ecf3cf27-e370-4cc5-86a4-628206277f58/0e6b288a-4b38-488e-b038-c06265dff781"
-					(reference "J5")
+					(reference "J6")
 					(unit 1)
 				)
@@
 			)
 		)
-		(property "Description" "Resistor"
+		(property "Description" ""
 			(at 129.54 101.6 0)
 			(effects
