File: KiCad/main_pcb/crystal.kicad_sch (KiCad schematic)
At the start: 3 parts, among them Y1 Crystal_GND24

Commit message: chore: Adds 3D models to footprint, instead of adding manually when placing components :3
Parts:
- Y1: private (none) -> KLC_S4.1
Changed lines of the file:
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@@
+			)
+		)
+		(property private "KLC_S3.3" "The rectangle is not a symbol body but a graphical element"
+			(at 120.65 101.6 0)
+			(effects
+				(font
+					(size 1.27 1.27)
+				)
+				(hide yes)
+			)
+		)
+		(property private "KLC_S4.1" "Some pins are on 50mil grid to make the symbol small"
+			(at 120.65 104.14 0)
+			(effects
+				(font
+					(size 1.27 1.27)
+				)
+				(hide yes)
 			)
 		)

Commit message: chore
Parts:
- Y1: private KLC_S4.1 -> (none)
- renumbered C11 to C13, C12 to C15
Changed lines of the file:
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@@
 		(on_board yes)
 		(dnp no)
-		(property "Reference" "C12"
+		(property "Reference" "C15"
 			(at 103.124 92.964 0)
 			(effects
@@
 			)
 		)
-		(property "Description" "Unpolarized capacitor"
+		(property "Description" ""
 			(at 110.49 93.98 0)
 			(effects
@@
 			(project "main_pcb"
 				(path "/ecf3cf27-e370-4cc5-86a4-628206277f58/4c1a0284-1742-4ed4-9190-6f37324df6a7"
-					(reference "C12")
+					(reference "C15")
 					(unit 1)
 				)
@@
 		(on_board yes)
 		(dnp no)
-		(property "Reference" "C11"
+		(property "Reference" "C13"
 			(at 132.334 92.964 0)
 			(effects
@@
 			)
 		)
-		(property "Description" "Unpolarized capacitor"
+		(property "Description" ""
 			(at 129.54 93.98 0)
 			(effects
@@
 			(project "main_pcb"
 				(path "/ecf3cf27-e370-4cc5-86a4-628206277f58/4c1a0284-1742-4ed4-9190-6f37324df6a7"
-					(reference "C11")
+					(reference "C13")
 					(unit 1)
 				)
@@
 			)
 		)
-		(property "Description" "Four pin crystal, GND on pins 2 and 4"
+		(property "Description" ""
 			(at 120.65 88.9 0)
 			(effects
@@
 			(effects
 				(font
-					(size 1.27 1.27)
-				)
-				(hide yes)
-			)
-		)
-		(property private "KLC_S3.3" "The rectangle is not a symbol body but a graphical element"
-			(at 120.65 101.6 0)
-			(effects
-				(font
-					(size 1.27 1.27)
-				)
-				(hide yes)
-			)
-		)
-		(property private "KLC_S4.1" "Some pins are on 50mil grid to make the symbol small"
-			(at 120.65 104.14 0)
-			(effects
-				(font
