File: KiCad/main_pcb/crystal.kicad_sch (KiCad schematic)
At the start: 3 parts, among them Y1 Crystal_GND24

Commit message: feat(KiCad): Adds part reference and fetches version that was taken into account by 42Chips when ordering so I can fix errors on the matching production files for the current PCB. :)
Parts:
- C3, C4: value 22pF -> 12pF; LCSC (none) -> C107034
- Y1: LCSC (none) -> C13738
Changed lines of the file:
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@@
 			)
 		)
-		(property "Value" "22pF"
+		(property "Value" "12pF"
 			(at 103.124 95.504 0)
 			(effects
@@
 		)
 		(property "Description" "Unpolarized capacitor"
+			(at 110.49 93.98 0)
+			(effects
+				(font
+					(size 1.27 1.27)
+				)
+				(hide yes)
+			)
+		)
+		(property "KLC_S3.3" ""
+			(at 110.49 93.98 0)
+			(effects
+				(font
+					(size 1.27 1.27)
+				)
+				(hide yes)
+			)
+		)
+		(property "KLC_S4.1" ""
+			(at 110.49 93.98 0)
+			(effects
+				(font
+					(size 1.27 1.27)
+				)
+				(hide yes)
+			)
+		)
+		(property "LCSC" "C107034"
 			(at 110.49 93.98 0)
 			(effects
@@
 			)
 		)
-		(property "Value" "22pF"
+		(property "Value" "12pF"
 			(at 132.334 95.504 0)
 			(effects
@@
 		)
 		(property "Description" "Unpolarized capacitor"
+			(at 129.54 93.98 0)
+			(effects
+				(font
+					(size 1.27 1.27)
+				)
+				(hide yes)
+			)
+		)
+		(property "KLC_S3.3" ""
+			(at 129.54 93.98 0)
+			(effects
+				(font
+					(size 1.27 1.27)
+				)
+				(hide yes)
+			)
+		)
+		(property "KLC_S4.1" ""
+			(at 129.54 93.98 0)
+			(effects
+				(font
+					(size 1.27 1.27)
+				)
+				(hide yes)
+			)
+		)
+		(property "LCSC" "C107034"
 			(at 129.54 93.98 0)
 			(effects
@@
 			(effects
 				(font
+					(size 1.27 1.27)
+				)
+				(hide yes)
+			)
+		)
+		(property "LCSC" "C13738"
+			(at 120.65 88.9 0)
+			(effects
+				(font

Commit message: Main PCB v2 (#51)
* feat(schematic & pcb): Switches to 2 rows header for keyboard connection

* feat(pcb): Keeps working on version 2 of main PCB

* feat(PCB): Continues work on PCB v2.

* feat(PCB): Continues work

* feat(PCB): Continues work

* feat(pcb): Workinonit

* feat(footprints): Adds homebrew USB-C

* chore(migration): Migrates to homebrew symbols for PCB.

* feat(footprints): Reworking footprints to allow hand-soldering

* feat(pcb): I think that's about right

* feat(pcb): Should be a-ok

* feat(PCB): Adds two pins header for LED Backlight

* feat(pcb): Uses new footprint for Male Header 2x13

* feat(3D models): Adds 3D models to PCB

* feat(schematic): Changes LED's resistor values from 330 ohms to 1k ohms.

* feat(3D models): Adds 3D model for push button switch

* feat(pcb): Adds all the remaning 3D models

* chore: Adds 3D models to footprint, instead of adding manually when placing components :3

* chore

* feat(sourcing): Changes Main PCB <-> Keyboard PCB connectors to something in stock

* chore

* chore

* chore

---------

Co-authored-by: Madeline Wolff <git@firmaments.anonaddy.com>
Parts:
- C13: renamed from C4; footprint Capacitor_SMD:C_0603_1608Metric_Pad1.08x0.95mm_HandSolder -> Lilibrary:Capacitor_0603
- C15: renamed from C3; footprint Capacitor_SMD:C_0603_1608Metric_Pad1.08x0.95mm_HandSolder -> Lilibrary:Capacitor_0603
- Y1: footprint Crystal:Crystal_SMD_3225-4Pin_3.2x2.5mm_HandSoldering -> Lilibrary:Crystal_3225; private KLC_S4.1 -> (none)
Changed lines of the file:
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@@
 		(on_board yes)
 		(dnp no)
-		(property "Reference" "C3"
+		(property "Reference" "C15"
 			(at 103.124 92.964 0)
 			(effects
@@
 			)
 		)
-		(property "Footprint" "Capacitor_SMD:C_0603_1608Metric_Pad1.08x0.95mm_HandSolder"
+		(property "Footprint" "Lilibrary:Capacitor_0603"
 			(at 109.5248 90.17 0)
 			(effects
@@
 			)
 		)
-		(property "Description" "Unpolarized capacitor"
+		(property "Description" ""
 			(at 110.49 93.98 0)
 			(effects
@@
 			(project "main_pcb"
 				(path "/ecf3cf27-e370-4cc5-86a4-628206277f58/4c1a0284-1742-4ed4-9190-6f37324df6a7"
-					(reference "C3")
+					(reference "C15")
 					(unit 1)
 				)
@@
 		(on_board yes)
 		(dnp no)
-		(property "Reference" "C4"
+		(property "Reference" "C13"
 			(at 132.334 92.964 0)
 			(effects
@@
 			)
 		)
-		(property "Footprint" "Capacitor_SMD:C_0603_1608Metric_Pad1.08x0.95mm_HandSolder"
+		(property "Footprint" "Lilibrary:Capacitor_0603"
 			(at 128.5748 90.17 0)
 			(effects
@@
 			)
 		)
-		(property "Description" "Unpolarized capacitor"
+		(property "Description" ""
 			(at 129.54 93.98 0)
 			(effects
@@
 			(project "main_pcb"
 				(path "/ecf3cf27-e370-4cc5-86a4-628206277f58/4c1a0284-1742-4ed4-9190-6f37324df6a7"
-					(reference "C4")
+					(reference "C13")
 					(unit 1)
 				)
@@
 			)
 		)
-		(property "Footprint" "Crystal:Crystal_SMD_3225-4Pin_3.2x2.5mm_HandSoldering"
+		(property "Footprint" "Lilibrary:Crystal_3225"
 			(at 120.65 88.9 0)
 			(effects
@@
 			)
 		)
-		(property "Description" "Four pin crystal, GND on pins 2 and 4"
+		(property "Description" ""
 			(at 120.65 88.9 0)
 			(effects
 				(font
-					(size 1.27 1.27)
-				)
-				(hide yes)
-			)
-		)
-		(property private "KLC_S3.3" "The rectangle is not a symbol body but a graphical element"
-			(at 120.65 101.6 0)
-			(show_name yes)
-			(effects
-				(font
-					(size 1.27 1.27)
-				)
-				(hide yes)
-			)
-		)
-		(property private "KLC_S4.1" "Some pins are on 50mil grid to make the symbol small"
-			(at 120.65 104.14 0)
-			(show_name yes)
-			(effects
-				(font
