File: kicad-keyboard-withlib/keyboard/keyboard.kicad_sch (KiCad schematic)
At the start: 45 parts, among them SW1 SW_Push, SW10 SW_Push, SW11 SW_Push, SW12 SW_Push, SW13 SW_Push, SW14 SW_Push, SW15 SW_Push, SW16 SW_Push, SW17 SW_Push, SW18 SW_Push, SW19 SW_Push, SW2 SW_Push, SW20 SW_Push, SW21 SW_Push, SW22 SW_Push, SW23 SW_Push, SW24 SW_Push, SW25 SW_Push, SW26 SW_Push, SW27 SW_Push, SW28 SW_Push, SW29 SW_Push, SW3 SW_Push, SW30 SW_Push, SW31 SW_Push, SW32 SW_Push, SW33 SW_Push, SW34 SW_Push, SW35 SW_Push, SW36 SW_Push, SW37 SW_Push, SW38 SW_Push, SW4 SW_Push, SW41 RotaryEncoder_Switch, SW42 SW_Wuerth_450301014042, SW5 SW_Push, SW6 SW_Push, SW7 SW_Push, SW8 SW_Push, SW9 SW_Push, U2 MCP23017_SO

Commit message: mid pcb commit in case of a kernel panic
Connections:
- net at SW42.1 (B): now also P1.18 (SLD_SW); no longer P1.17 (SLD_SW)
- net at SW42.2 (C): now also P1.17 (SLD_SW); no longer P1.19 (SLD_SW)
- net at SW42.3 (A): now also P1.19 (SLD_SW); no longer P1.18 (SLD_SW)
Changed lines of the file:
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@@
+	(wire
+		(pts
+			(xy 191.77 62.23) (xy 191.77 59.69)
+		)
+		(stroke
+			(width 0)
+			(type default)
+		)
+	)
 	(wire
 		(pts
@@
 	(wire
 		(pts
-			(xy 201.93 46.99) (xy 162.56 46.99)
-		)
-		(stroke
-			(width 0)
-			(type default)
-		)
-	)
-	(wire
-		(pts
 			(xy 144.78 43.18) (xy 124.46 43.18)
 		)
@@
 	(wire
 		(pts
+			(xy 162.56 57.15) (xy 181.61 57.15)
+		)
+		(stroke
+			(width 0)
+			(type default)
+		)
+	)
+	(wire
+		(pts
 			(xy 157.48 31.75) (xy 157.48 27.94)
 		)
@@
 	(wire
 		(pts
-			(xy 160.02 57.15) (xy 181.61 57.15)
-		)
-		(stroke
-			(width 0)
-			(type default)
-		)
-	)
-	(wire
-		(pts
 			(xy 121.92 31.75) (xy 121.92 27.94)
 		)
@@
 	(wire
 		(pts
-			(xy 160.02 27.94) (xy 160.02 57.15)
-		)
-		(stroke
-			(width 0)
-			(type default)
-		)
-	)
-	(wire
-		(pts
 			(xy 20.32 127) (xy 20.32 132.08)
 		)
@@
 	(wire
 		(pts
+			(xy 160.02 62.23) (xy 191.77 62.23)
+		)
+		(stroke
+			(width 0)
+			(type default)
+		)
+	)
+	(wire
+		(pts
 			(xy 132.08 27.94) (xy 132.08 36.83)
 		)
@@
 	(wire
 		(pts
-			(xy 201.93 54.61) (xy 191.77 54.61)
-		)
-		(stroke
-			(width 0)
-			(type default)
-		)
-	)
-	(wire
-		(pts
 			(xy 20.32 102.87) (xy 20.32 107.95)
 		)
@@
 	(wire
 		(pts
-			(xy 201.93 46.99) (xy 201.93 54.61)
-		)
-		(stroke
-			(width 0)
-			(type default)
-		)
-	)
-	(wire
-		(pts
 			(xy 144.78 107.95) (xy 144.78 102.87)
 		)
@@
 	(wire
 		(pts
-			(xy 204.47 44.45) (xy 204.47 59.69)
-		)
-		(stroke
-			(width 0)
-			(type default)
-		)
-	)
-	(wire
-		(pts
 			(xy 68.58 179.07) (xy 83.82 179.07)
 		)
@@
 	(wire
 		(pts
+			(xy 191.77 54.61) (xy 204.47 54.61)
+		)
+		(stroke
+			(width 0)
+			(type default)
+		)
+	)
+	(wire
+		(pts
 			(xy 99.06 179.07) (xy 114.3 179.07)
 		)
@@
 	(wire
 		(pts
+			(xy 204.47 44.45) (xy 204.47 54.61)
+		)
+		(stroke
+			(width 0)
+			(type default)
+		)
+	)
+	(wire
+		(pts
 			(xy 142.24 27.94) (xy 142.24 41.91)
 		)
@@
 	(wire
 		(pts
-			(xy 204.47 59.69) (xy 191.77 59.69)
-		)
-		(stroke
-			(width 0)
-			(type default)
-		)
-	)
-	(wire
-		(pts
 			(xy 186.69 93.98) (xy 186.69 63.5)
 		)
@@
 	(wire
 		(pts
+			(xy 160.02 27.94) (xy 160.02 62.23)
+		)
+		(stroke
+			(width 0)
+			(type default)
+		)
+	)
+	(wire
+		(pts
 			(xy 99.06 154.94) (xy 99.06 149.86)
 		)
@@
 	(wire
 		(pts
-			(xy 162.56 46.99) (xy 162.56 27.94)
-		)
-		(stroke
+			(xy 162.56 27.94) (xy 162.56 57.15)
+		)
+		(stroke

Commit message: fix: VCC netclass resized
Parts:
- removed SW42: SW_Wuerth_450301014042, Button_Switch_THT:SW_Slide-03_Wuerth-WS-SLTV_10x2.5x6.4_P2.54mm, symbol Switch:SW_Wuerth_450301014042
- added SW39: SW_Slide_DPDT, Button_Switch_THT:SW_CK_JS202011CQN_DPDT_Straight, symbol Switch:SW_Slide_DPDT
Connections:
- net at P1.18 (SLD_SW): now also SW39.2 (B)
- net at P1.17 (SLD_SW): now also SW39.1 (A)
- net at P1.19 (SLD_SW): now also SW39.3 (C)
Changed lines of the file:
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@@
 	(wire
 		(pts
+			(xy 175.26 41.91) (xy 175.26 44.45)
+		)
+		(stroke
+			(width 0)
+			(type default)
+		)
+	)
+	(wire
+		(pts
 			(xy 129.54 154.94) (xy 129.54 149.86)
 		)
@@
 	(wire
 		(pts
-			(xy 160.02 132.08) (xy 160.02 127)
+			(xy 162.56 39.37) (xy 180.34 39.37)
 		)
 		(stroke
@@
 	(wire
 		(pts
-			(xy 196.85 85.09) (xy 196.85 86.36)
+			(xy 160.02 132.08) (xy 160.02 127)
 		)
 		(stroke
@@
 	(wire
 		(pts
-			(xy 53.34 107.95) (xy 53.34 102.87)
+			(xy 196.85 85.09) (xy 196.85 86.36)
 		)
 		(stroke
@@
 	(wire
 		(pts
-			(xy 149.86 44.45) (xy 154.94 44.45)
+			(xy 53.34 107.95) (xy 53.34 102.87)
 		)
 		(stroke
@@
 	(wire
 		(pts
-			(xy 191.77 62.23) (xy 191.77 59.69)
+			(xy 149.86 44.45) (xy 154.94 44.45)
 		)
 		(stroke
@@
 	(wire
 		(pts
-			(xy 162.56 57.15) (xy 181.61 57.15)
-		)
-		(stroke
-			(width 0)
-			(type default)
-		)
-	)
-	(wire
-		(pts
 			(xy 157.48 31.75) (xy 157.48 27.94)
 		)
@@
 	(wire
 		(pts
+			(xy 160.02 41.91) (xy 175.26 41.91)
+		)
+		(stroke
+			(width 0)
+			(type default)
+		)
+	)
+	(wire
+		(pts
 			(xy 121.92 31.75) (xy 121.92 27.94)
 		)
@@
 	(wire
 		(pts
+			(xy 180.34 39.37) (xy 180.34 44.45)
+		)
+		(stroke
+			(width 0)
+			(type default)
+		)
+	)
+	(wire
+		(pts
 			(xy 20.32 113.03) (xy 20.32 127)
 		)
@@
 	(wire
 		(pts
-			(xy 139.7 27.94) (xy 139.7 40.64)
+			(xy 165.1 36.83) (xy 185.42 36.83)
 		)
 		(stroke
@@
 	(wire
 		(pts
-			(xy 154.94 44.45) (xy 154.94 102.87)
+			(xy 139.7 27.94) (xy 139.7 40.64)
 		)
 		(stroke
@@
 	(wire
 		(pts
-			(xy 20.32 127) (xy 20.32 132.08)
+			(xy 154.94 44.45) (xy 154.94 102.87)
 		)
 		(stroke
@@
 	(wire
 		(pts
-			(xy 165.1 44.45) (xy 204.47 44.45)
+			(xy 20.32 127) (xy 20.32 132.08)
 		)
 		(stroke
@@
 	(wire
 		(pts
-			(xy 160.02 62.23) (xy 191.77 62.23)
+			(xy 160.02 27.94) (xy 160.02 41.91)
 		)
 		(stroke
@@
 	(wire
 		(pts
-			(xy 191.77 54.61) (xy 204.47 54.61)
-		)
-		(stroke
-			(width 0)
-			(type default)
-		)
-	)
-	(wire
-		(pts
 			(xy 99.06 179.07) (xy 114.3 179.07)
 		)
@@
 	(wire
 		(pts
-			(xy 165.1 27.94) (xy 165.1 44.45)
+			(xy 142.24 27.94) (xy 142.24 41.91)
 		)
 		(stroke
@@
 	(wire
 		(pts
-			(xy 204.47 44.45) (xy 204.47 54.61)
+			(xy 185.42 36.83) (xy 185.42 44.45)
 		)
 		(stroke
@@
 	(wire
 		(pts
-			(xy 142.24 27.94) (xy 142.24 41.91)
+			(xy 17.78 135.89) (xy 20.32 135.89)
 		)
 		(stroke
@@
 	(wire
 		(pts
-			(xy 17.78 135.89) (xy 20.32 135.89)
+			(xy 38.1 179.07) (xy 38.1 173.99)
 		)
 		(stroke
@@
 	(wire
 		(pts
-			(xy 38.1 179.07) (xy 38.1 173.99)
+			(xy 20.32 102.87) (xy 22.86 102.87)
 		)
 		(stroke
@@
 	(wire
 		(pts
-			(xy 20.32 102.87) (xy 22.86 102.87)
+			(xy 38.1 179.07) (xy 53.34 179.07)
 		)
 		(stroke
@@
 	(wire
 		(pts
-			(xy 38.1 179.07) (xy 53.34 179.07)
+			(xy 109.22 149.86) (xy 109.22 173.99)
 		)
 		(stroke
@@
 	(wire
 		(pts
-			(xy 109.22 149.86) (xy 109.22 173.99)
+			(xy 165.1 27.94) (xy 165.1 36.83)
 		)
 		(stroke
@@
 	(wire
 		(pts
+			(xy 162.56 27.94) (xy 162.56 39.37)
+		)
+		(stroke
+			(width 0)
+			(type default)
+		)
+	)
+	(wire
+		(pts
 			(xy 186.69 93.98) (xy 186.69 63.5)
 		)
@@
 	(wire
 		(pts
-			(xy 160.02 27.94) (xy 160.02 62.23)
-		)
-		(stroke
-			(width 0)
-			(type default)
-		)
-	)
-	(wire
-		(pts
 			(xy 99.06 154.94) (xy 99.06 149.86)
 		)
@@
 		)
 	)
-	(wire
-		(pts
-			(xy 162.56 27.94) (xy 162.56 57.15)
-		)
-		(stroke
-			(width 0)
-			(type default)
-		)
-	)
 	(symbol
 		(lib_id "Switch:SW_Push")
@@
 	)
 	(symbol
-		(lib_id "Switch:SW_Wuerth_450301014042")
-		(at 186.69 57.15 0)
-		(unit 1)
-		(exclude_from_sim no)
-		(in_bom yes)
-		(on_board yes)
-		(dnp no)
-		(fields_autoplaced yes)
-		(property "Reference" "SW42"
-			(at 186.69 48.26 0)
-			(effects
-				(font
-					(size 1.27 1.27)
-				)
-			)
-		)
-		(property "Value" "SW_Wuerth_450301014042"
-			(at 186.69 50.8 0)
-			(effects
-				(font
-					(size 1.27 1.27)
-				)
-			)
-		)
-		(property "Footprint" "Button_Switch_THT:SW_Slide-03_Wuerth-WS-SLTV_10x2.5x6.4_P2.54mm"
-			(at 186.69 67.31 0)
-			(effects
-				(font
-					(size 1.27 1.27)
-				)
-				(hide yes)
-			)
-		)
-		(property "Datasheet" "https://www.we-online.com/components/products/datasheet/450301014042.pdf"
-			(at 186.69 64.77 0)
-			(effects
-				(font
-					(size 1.27 1.27)
-				)
-				(hide yes)
-			)
-		)
-		(property "Description" "Switch slide, single pole double throw"
-			(at 186.69 57.15 0)
-			(effects
-				(font
-					(size 1.27 1.27)
-				)
-				(hide yes)
-			)
-		)
-		(pin "3"
-		)
-		(pin "1"
-		)
-		(pin "2"
-		)
-		(instances
-			(project ""
-				(path "/55764147-763c-452f-85b8-3be2d22c3190"
-					(reference "SW42")
-					(unit 1)
-				)
-			)
-		)
-	)
-	(symbol
 		(lib_id "Switch:SW_Push")
 		(at 88.9 102.87 0)
@@
 					(unit 1)
 				)
+			)
+		)
+	)
+	(symbol
+		(lib_id "Switch:SW_Slide_DPDT")
+		(at 180.34 49.53 90)
+		(mirror x)
+		(unit 1)
+		(exclude_from_sim no)
+		(in_bom yes)
+		(on_board yes)
+		(dnp no)
+		(property "Reference" "SW39"
+			(at 173.99 48.2599 90)
+			(effects
+				(font
+					(size 1.27 1.27)
+				)
+				(justify left)
+			)
+		)
+		(property "Value" "SW_Slide_DPDT"
+			(at 173.99 50.7999 90)
+			(effects
+				(font
+					(size 1.27 1.27)
+				)
+				(justify left)
+			)
+		)
+		(property "Footprint" "Button_Switch_THT:SW_CK_JS202011CQN_DPDT_Straight"
+			(at 175.26 63.5 0)
+			(effects
+				(font
+					(size 1.27 1.27)
+				)
+				(hide yes)
+			)
+		)
+		(property "Datasheet" "~"
+			(at 180.34 49.53 0)
+			(effects
+				(font
+					(size 1.27 1.27)
+				)
+				(hide yes)
+			)
+		)
+		(property "Description" "Slide Switch, dual pole double throw"
+			(at 180.34 49.53 0)
+			(effects
+				(font
+					(size 1.27 1.27)
+				)
+				(hide yes)
+			)
+		)
+		(pin "1"
+		)
+		(pin "5"
+		)
+		(pin "3"
+		)
+		(pin "2"
+		)
+		(pin "6"
+		)
+		(pin "4"
+		)
+		(instances
+			(project ""
+				(path "/55764147-763c-452f-85b8-3be2d22c3190"
+					(reference "SW39")
+					(unit 1)
+				)
