File: kicad-keyboard-withlib/keyboard/keyboard.kicad_sch (KiCad schematic)
At the start: 85 parts, among them SW1 SW_Push, SW10 SW_Push, SW11 SW_Push, SW12 SW_Push, SW13 SW_Push, SW14 SW_Push, SW15 SW_Push, SW16 SW_Push, SW17 SW_Push, SW18 SW_Push, SW19 SW_Push, SW2 SW_Push, SW20 SW_Push, SW21 SW_Push, SW22 SW_Push, SW23 SW_Push, SW24 SW_Push, SW25 SW_Push, SW26 SW_Push, SW27 SW_Push, SW28 SW_Push, SW29 SW_Push, SW3 SW_Push, SW30 SW_Push, SW31 SW_Push, SW32 SW_Push, SW33 SW_Push, SW34 SW_Push, SW35 SW_Push, SW36 SW_Push, SW37 SW_Push, SW38 SW_Push, SW39 SW_Slide_DPDT, SW4 SW_Push, SW5 SW_Push, SW6 SW_Push, SW7 SW_Push, SW8 SW_Push, SW9 SW_Push, U2 MCP23017_SO

Commit message: add: started the pcb with diode, add the 10k missing comments silkscreen
Parts:
- D1: renamed from U13; footprint (none) -> Lilyspad:diode
- D10: renamed from U4; footprint (none) -> Lilyspad:diode
- D11: renamed from U14; footprint (none) -> Lilyspad:diode
- D12: renamed from U15; footprint (none) -> Lilyspad:diode
- D13: renamed from U16; footprint (none) -> Lilyspad:diode
- D14: renamed from U17; footprint (none) -> Lilyspad:diode
- D15: renamed from U18; footprint (none) -> Lilyspad:diode
- D16: renamed from U19; footprint (none) -> Lilyspad:diode
- D17: renamed from U20; footprint (none) -> Lilyspad:diode
- D18: renamed from U21; footprint (none) -> Lilyspad:diode
- D19: renamed from U22; footprint (none) -> Lilyspad:diode
- D2: renamed from U12; footprint (none) -> Lilyspad:diode
- D20: renamed from U23; footprint (none) -> Lilyspad:diode
- D21: renamed from U33; footprint (none) -> Lilyspad:diode
- D22: renamed from U32; footprint (none) -> Lilyspad:diode
- D23: renamed from U31; footprint (none) -> Lilyspad:diode
- D24: renamed from U30; footprint (none) -> Lilyspad:diode
- D25: renamed from U29; footprint (none) -> Lilyspad:diode
- D26: renamed from U28; footprint (none) -> Lilyspad:diode
- D27: renamed from U27; footprint (none) -> Lilyspad:diode
- D28: renamed from U26; footprint (none) -> Lilyspad:diode
- D29: renamed from U25; footprint (none) -> Lilyspad:diode
- D3: renamed from U11; footprint (none) -> Lilyspad:diode
- D30: renamed from U24; footprint (none) -> Lilyspad:diode
- D31: renamed from U34; footprint (none) -> Lilyspad:diode
- D32: renamed from U35; footprint (none) -> Lilyspad:diode
- D33: renamed from U36; footprint (none) -> Lilyspad:diode
- D34: renamed from U37; footprint (none) -> Lilyspad:diode
- D35: renamed from U38; footprint (none) -> Lilyspad:diode
- D36: renamed from U39; footprint (none) -> Lilyspad:diode
- D37: renamed from U40; footprint (none) -> Lilyspad:diode
- D38: renamed from U41; footprint (none) -> Lilyspad:diode
- D4: renamed from U10; footprint (none) -> Lilyspad:diode
- D5: renamed from U9; footprint (none) -> Lilyspad:diode
- D6: renamed from U8; footprint (none) -> Lilyspad:diode
- D7: renamed from U7; footprint (none) -> Lilyspad:diode
- D8: renamed from U6; footprint (none) -> Lilyspad:diode
- D9: renamed from U5; footprint (none) -> Lilyspad:diode
- U2: footprint Lilyspad:MCP23017 -> Package_SO:SOIC-28W_7.5x17.9mm_P1.27mm
