File: KiCad/main_pcb/main_pcb/crystal.kicad_sch (KiCad schematic)
At the start: 3 parts, among them Y1 Crystal_GND24

Commit message: feat(schematic): Assigns footprints to symbols
Parts:
- C3, C4: footprint (none) -> Capacitor_SMD:C_0603_1608Metric_Pad1.08x0.95mm_HandSolder
- Y1: footprint (none) -> Crystal:Crystal_SMD_3225-4Pin_3.2x2.5mm_HandSoldering
Changed lines of the file:
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@@
 			)
 		)
-		(property "Footprint" ""
+		(property "Footprint" "Capacitor_SMD:C_0603_1608Metric_Pad1.08x0.95mm_HandSolder"
 			(at 109.5248 90.17 0)
 			(effects
@@
 			)
 		)
-		(property "Footprint" ""
+		(property "Footprint" "Capacitor_SMD:C_0603_1608Metric_Pad1.08x0.95mm_HandSolder"
 			(at 128.5748 90.17 0)
 			(effects
@@
 		(dnp no)
 		(fields_autoplaced yes)
-		(property "Reference" "#PWR018"
+		(property "Reference" "#PWR017"
 			(at 120.65 106.68 0)
 			(effects
@@
 			(project "main_pcb"
 				(path "/ecf3cf27-e370-4cc5-86a4-628206277f58/4c1a0284-1742-4ed4-9190-6f37324df6a7"
-					(reference "#PWR018")
+					(reference "#PWR017")
 					(unit 1)
 				)
@@
 			)
 		)
-		(property "Footprint" ""
+		(property "Footprint" "Crystal:Crystal_SMD_3225-4Pin_3.2x2.5mm_HandSoldering"
 			(at 120.65 88.9 0)
 			(effects

Commit message: feat(PCB): Updates PCB layout after Christian's review, thansk a lot Christian :) !
Parts:
- C3, C4: value 33pF -> 22pF
Other:
- note added: "Check capacitor value for Lab's crystals"
Changed lines of the file:
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@@
 	(generator_version "9.0")
 	(paper "A4")
+	(text "Check capacitor value for Lab's crystals\n"
+		(exclude_from_sim no)
+		(at 93.98 103.632 0)
+		(effects
+			(font
+				(size 1.27 1.27)
+			)
+		)
+	)
 	(junction
 		(at 129.54 88.9)
@@
 			)
 		)
-		(property "Value" "33pF"
+		(property "Value" "22pF"
 			(at 103.124 95.504 0)
 			(effects
@@
 			)
 		)
-		(property "Value" "33pF"
+		(property "Value" "22pF"
 			(at 132.334 95.504 0)
 			(effects
