File: KiCad/main_pcb.bak/main_pcb.kicad_sch (KiCad schematic)
At the start: 18 parts, among them J1 1x21 Header, J3 1x6 Header, U1 ATmega 2560

Commit message: Maddie/main pcb refactor (#39)
* feat(PCB Layout): Refactors Main PCB layout to achieve smaller form factor and adds JLCPCB constraints.

* feat(symbols): Adds 4pin crystal symbols and adds it to schematic

* feat(schematic): Connects C2 and C3 to the crystal

* feat(schematic): Revamps fully the circuit schematic

* feat(schematic): Assigns footprints to symbols

* feat(pcb): Alternative first draft

* feat(pcb): Second draft

* feat(pdf): Updates schematic PDF

* feat(pdf): Updates schematic PDF

* chore(migration): Puts old layout in main_pcb.bak/ and new layout to main_pcb/

* feat(PCB): Updates PCB layout after Christian's review, thansk a lot Christian :) !
Parts:
- added C5: 100nF, Capacitor_SMD:C_0201_0603Metric_Pad0.64x0.40mm_HandSolder, symbol Lily's Pad:Capacitor
- added J2: ~, Connector_JST:JST_XH_B10B-XH-A_1x10_P2.50mm_Vertical, symbol Lily's Pad:2X5_Header
- C1, C2, C3, C4: footprint Capacitor_SMD:C_0603_1608Metric_Pad1.08x0.95mm_HandSolder -> Capacitor_SMD:C_0201_0603Metric_Pad0.64x0.40mm_HandSolder
- J1: value 1x21 Header -> ~; footprint Lilibrary:1x21 Header -> (none); symbol Lily's Pad:1x21 Header -> Lily's Pad:Header_21
- R1, R2, R3, R4, R5: footprint Resistor_SMD:R_0603_1608Metric_Pad0.98x0.95mm_HandSolder -> Resistor_SMD:R_0201_0603Metric_Pad0.64x0.40mm_HandSolder
- U1: value ATmega 2560 -> ~
- Y1: footprint Crystal:Crystal_SMD_0603-4Pin_6.0x3.5mm_HandSoldering -> Crystal:Crystal_SMD_ECS_CSM3X-2Pin_7.6x4.1mm
Connections:
- net GND: now also C5.1, C5.2, J2.10, J2.2; no longer Y1.2 (G), Y1.4 (G)
- net VCC: now also J2.4, J2.7
- net uC_Reset: now also J2.6
- net at C3.2: now also Y1.2; no longer Y1.1
- net at C2.2: now also Y1.1; no longer Y1.3
- net TDI: now reaches U1.90 (PF7)
- net TDI: now also J2.9
- net TDO: now reaches U1.91 (PF6)
- net TDO: now also J2.3
- net TMS: now reaches U1.92 (PF5)
- net TMS: now also J2.5
- net TCK: now reaches U1.93 (PF4)
- net TCK: now also J2.1
- no-connect marks 53 -> 50
Other:
- moved on the sheet: C3
