File: kicad-keyboard/keyboard/keyboard.kicad_pcb (KiCad board)
At the start: 2 copper layers, 149.1 x 131.9 mm, 96 parts, among them SW1 SW_Push, SW10 SW_Push, SW11 SW_Push, SW12 SW_Push, SW13 SW_Push, SW14 SW_Push, SW15 SW_Push, SW16 SW_Push, SW17 SW_Push, SW18 SW_Push, SW19 SW_Push, SW2 SW_Push, SW20 SW_Push, SW21 SW_Push, SW22 SW_Push, SW23 SW_Push, SW24 SW_Push, SW25 SW_Push, SW26 SW_Push, SW27 SW_Push, SW28 SW_Push, SW29 SW_Push, SW3 SW_Push, SW30 SW_Push, SW31 SW_Push, SW32 SW_Push, SW33 SW_Push, SW34 SW_Push, SW35 SW_Push, SW36 SW_Push, SW37 SW_Push, SW38 SW_Push, SW39 SW_Slide_DPDT, SW4 SW_Push, SW5 SW_Push, SW6 SW_Push, SW7 SW_Push, SW8 SW_Push, SW9 SW_Push, U2 MCP23017_SO

Commit message: add: fix some i2c thing
Parts:
- removed U2: MCP23017_SO, Package_SO:SOIC-28W_7.5x17.9mm_P1.27mm
- added MCP1: ~, Lilyspad:MCP23017, F.Cu at (148.6, 149.9)
Routing:
- net GND: track 8.99 -> 11.4 mm
- net Net-(MCP1-SCK): track 197.8 -> 199.7 mm
