File: hardware/kicad-keyboard/keyboard/keyboard.kicad_pcb (KiCad board)
At the start: 2 copper layers, 149.1 x 131.9 mm, 96 parts, among them SW1 SW_Push, SW10 SW_Push, SW11 SW_Push, SW12 SW_Push, SW13 SW_Push, SW14 SW_Push, SW15 SW_Push, SW16 SW_Push, SW17 SW_Push, SW18 SW_Push, SW19 SW_Push, SW2 SW_Push, SW20 SW_Push, SW21 SW_Push, SW22 SW_Push, SW23 SW_Push, SW24 SW_Push, SW25 SW_Push, SW26 SW_Push, SW27 SW_Push, SW28 SW_Push, SW29 SW_Push, SW3 SW_Push, SW30 SW_Push, SW31 SW_Push, SW32 SW_Push, SW33 SW_Push, SW34 SW_Push, SW35 SW_Push, SW36 SW_Push, SW37 SW_Push, SW38 SW_Push, SW39 SW_Slide_DPDT, SW4 SW_Push, SW5 SW_Push, SW6 SW_Push, SW7 SW_Push, SW8 SW_Push, SW9 SW_Push

Commit message: fix: Reannotates schematic components
Parts:
- removed D1: LED, Lilyspad:led
- removed MCP23017: ~, Lilyspad:MCP23017
- added MCP1: ~, Lilyspad:MCP23017, F.Cu at (148.7, 149.6)
- renumbered D9 to D10, D10 to D11, D11 to D12, D12 to D13, D13 to D14, D14 to D15, D15 to D16, D16 to D17, D17 to D18, D18 to D19, D1 to D2, D19 to D20, D20 to D21, D21 to D22, D22 to D23, D23 to D24, D24 to D25, D25 to D26, D26 to D27, D27 to D28, D28 to D29, D2 to D3, D29 to D30, D30 to D31, D31 to D32, D32 to D33, D33 to D34, D34 to D35, D35 to D36, D36 to D37, D37 to D38, D38 to D39, D3 to D4, D4 to D5, D5 to D6, D6 to D7, D7 to D8, D8 to D9, R4 to R1, R3 to R2, R2 to R3, R1 to R4, SW39 to SW1, SW8 to SW10, SW9 to SW11, SW10 to SW12, SW11 to SW13, SW12 to SW14, SW13 to SW15, SW14 to SW16, SW15 to SW17, SW16 to SW18, SW17 to SW19, SW40 to SW2, SW18 to SW20, SW19 to SW21, SW20 to SW22, SW21 to SW23, SW22 to SW24, SW23 to SW25, SW24 to SW26, SW25 to SW27, SW26 to SW28, SW27 to SW29, SW1 to SW3, SW28 to SW30, SW29 to SW31, SW30 to SW32, SW31 to SW33, SW32 to SW34, SW33 to SW35, SW34 to SW36, SW35 to SW37, SW36 to SW38, SW37 to SW39, SW2 to SW4, SW38 to SW40, SW3 to SW5, SW4 to SW6, SW5 to SW7, SW6 to SW8, SW7 to SW9
Routing:
- net Net-(U1-R4): track 257.5 -> 0.00 mm
- net Net-(U1-R3): track 249.4 -> 0.00 mm
- net VCC: track 204.9 -> 0.00 mm
- net Net-(MCP1-SDA): track 208.5 -> 15.7 mm
- net Net-(MCP1-SCK): track 199.7 -> 12.0 mm
- net Net-(U1-R2): track 172.7 -> 0.00 mm
- net Net-(U1-C8): track 167.0 -> 0.00 mm, vias 4 -> 0
- net Net-(U1-R1): track 146.6 -> 0.00 mm
- net Net-(U1-C10): track 128.4 -> 0.00 mm, vias 2 -> 0
- net Net-(U1-C7): track 127.4 -> 0.00 mm, vias 6 -> 0
- net Net-(U1-C9): track 122.1 -> 0.00 mm, vias 4 -> 0
- net Net-(U1-C6): track 120.3 -> 0.00 mm, vias 6 -> 0
- net Net-(U1-C5): track 106.8 -> 0.00 mm, vias 6 -> 0
- net Net-(U1-C4): track 106.1 -> 0.00 mm, vias 6 -> 0
- net Net-(U1-C1): track 103.4 -> 0.00 mm, vias 6 -> 0
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
Commit message: fix: Reworks keyboard PCB
Parts:
- added D1: ~, Lilyspad:led, F.Cu at (162.8, 80.3)
- moved D30 13.0 mm to (133.1, 122.4)
- moved D38 12.3 mm to (122.1, 143.0)
- moved D21 11.5 mm to (143.8, 100.6)
- moved D11 11.3 mm to (144.4, 79.4)
- moved R4 0.75 mm to (152.2, 137.0)
Routing:
- net Net-(U1-R4): track 0.00 -> 270.2 mm
- net Net-(U1-R3): track 0.00 -> 251.7 mm
- net VCC: track 0.00 -> 236.8 mm, vias 2 -> 0
- net Net-(U1-C8): track 0.00 -> 196.1 mm, vias 0 -> 6
- net Net-(MCP1-SDA): track 15.7 -> 205.6 mm, vias 0 -> 2
- net Net-(MCP1-SCK): track 12.0 -> 196.3 mm, vias 0 -> 2
- net Net-(U1-R2): track 0.00 -> 182.5 mm
- net Net-(U1-C10): track 0.00 -> 178.2 mm, vias 0 -> 2
- net Net-(U1-R1): track 0.00 -> 167.1 mm
- net Net-(U1-C7): track 0.00 -> 161.2 mm, vias 0 -> 6
- net Net-(U1-C6): track 0.00 -> 154.0 mm, vias 0 -> 6
- net Net-(U1-C9): track 0.00 -> 149.8 mm, vias 0 -> 4
- net Net-(U1-C5): track 0.00 -> 143.2 mm, vias 0 -> 6
- net Net-(U1-C4): track 0.00 -> 136.5 mm, vias 0 -> 6
- net Net-(U1-C2): track 0.00 -> 125.2 mm, vias 0 -> 6
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
Commit message: chore: keyboard PCB review done
Parts:
- added G***: LOGO, LOGO, F.Cu at (99.7, 53.1)
- moved G*** 65.4 mm to (54.4, 72.2)
Routing:
- net VCC: track 236.8 -> 237.9 mm

Commit message: fix: Numerotation fix
Parts:
- renumbered D2 to D1, D11 to D10, D31 to D11, D1 to D12, D12 to D13, D13 to D14, D14 to D15, D15 to D16, D16 to D17, D17 to D18, D18 to D19, D3 to D2, D19 to D20, D20 to D21, D21 to D22, D39 to D23, D22 to D24, D23 to D25, D24 to D26, D25 to D27, D26 to D28, D27 to D29, D4 to D3, D28 to D30, D30 to D31, D29 to D32, D32 to D33, D33 to D34, D34 to D35, D35 to D36, D36 to D37, D37 to D38, D38 to D39, D5 to D4, D6 to D5, D7 to D6, D8 to D7, D9 to D8, D10 to D9, M4 to M3, M3 to M4, R4 to R2, R2 to R4, SW11 to SW10, SW12 to SW11, SW32 to SW12, SW3 to SW2, SW40 to SW23, SW2 to SW24, SW23 to SW25, SW24 to SW26, SW25 to SW27, SW26 to SW28, SW27 to SW29, SW4 to SW3, SW28 to SW30, SW29 to SW31, SW30 to SW32, SW31 to SW33, SW33 to SW34, SW34 to SW35, SW35 to SW36, SW36 to SW37, SW37 to SW38, SW38 to SW39, SW5 to SW4, SW39 to SW40, SW6 to SW5, SW7 to SW6, SW8 to SW7, SW9 to SW8, SW10 to SW9
