File: hardware/kicad-keyboard/keyboard/keyboard.kicad_pcb (KiCad board)
At the start: 2 copper layers, 149.1 x 131.9 mm, 96 parts, among them SW1 SW_Push, SW10 SW_Push, SW11 SW_Push, SW12 SW_Push, SW13 SW_Push, SW14 SW_Push, SW15 SW_Push, SW16 SW_Push, SW17 SW_Push, SW18 SW_Push, SW19 SW_Push, SW2 SW_Push, SW20 SW_Push, SW21 SW_Push, SW22 SW_Push, SW23 SW_Push, SW24 SW_Push, SW25 SW_Push, SW26 SW_Push, SW27 SW_Push, SW28 SW_Push, SW29 SW_Push, SW3 SW_Push, SW30 SW_Push, SW31 SW_Push, SW32 SW_Push, SW33 SW_Push, SW34 SW_Push, SW35 SW_Push, SW36 SW_Push, SW37 SW_Push, SW38 SW_Push, SW39 SW_Slide_DPDT, SW4 SW_Push, SW5 SW_Push, SW6 SW_Push, SW7 SW_Push, SW8 SW_Push, SW9 SW_Push

Commit message: Keyboard pcb fix (#74)
* fix: Fixes push button switch footprint pad assignation

* fix: Fixes rotary encoder footprint pad assignation

* fix: Reannotates schematic components

* fix: Reworks keyboard PCB

* chore: KiCad updates

* chore: keyboard PCB review done

* fix: Numerotation fix

* chore: Adds some 3D models
Parts:
- removed the D1 at (162.8, 74.8)
- removed MCP23017: ~, Lilyspad:MCP23017
- added D12: ~, Lilyspad:led, F.Cu at (162.8, 80.3)
- added G***: LOGO, LOGO, F.Cu at (99.7, 53.1)
- added MCP1: ~, Lilyspad:MCP23017, F.Cu at (148.7, 149.6)
- moved G*** 65.4 mm to (54.4, 72.2)
- moved D31 13.0 mm to (133.1, 122.4)
- moved D39 12.3 mm to (122.1, 143.0)
- moved D22 11.5 mm to (143.8, 100.6)
- moved D10 11.3 mm to (144.4, 79.4)
- moved R2 0.75 mm to (152.2, 137.0)
- renumbered D30 to D11, D11 to D13, D12 to D14, D13 to D15, D14 to D16, D15 to D17, D16 to D18, D17 to D19, D18 to D20, D19 to D21, D20 to D22, D38 to D23, D21 to D24, D22 to D25, D23 to D26, D24 to D27, D25 to D28, D26 to D29, D27 to D30, D29 to D31, D28 to D32, D31 to D33, D32 to D34, D33 to D35, D34 to D36, D35 to D37, D36 to D38, D37 to D39, M4 to M3, M3 to M4, R4 to R1, R1 to R2, R2 to R3, R3 to R4, SW39 to SW1, SW9 to SW10, SW10 to SW11, SW30 to SW12, SW11 to SW13, SW12 to SW14, SW13 to SW15, SW14 to SW16, SW15 to SW17, SW16 to SW18, SW17 to SW19, SW1 to SW2, SW18 to SW20, SW19 to SW21, SW20 to SW22, SW38 to SW23, SW40 to SW24, SW21 to SW25, SW22 to SW26, SW23 to SW27, SW24 to SW28, SW25 to SW29, SW2 to SW3, SW26 to SW30, SW27 to SW31, SW28 to SW32, SW29 to SW33, SW31 to SW34, SW32 to SW35, SW33 to SW36, SW34 to SW37, SW35 to SW38, SW36 to SW39, SW3 to SW4, SW37 to SW40, SW4 to SW5, SW5 to SW6, SW6 to SW7, SW7 to SW8, SW8 to SW9
Routing:
- net Net-(U1-C10): track 128.4 -> 178.2 mm
- net Net-(U1-C5): track 106.8 -> 143.2 mm
- net Net-(U1-C7): track 127.4 -> 161.2 mm
- net Net-(U1-C6): track 120.3 -> 154.0 mm
- net VCC: track 204.9 -> 237.9 mm, vias 2 -> 0
- net Net-(U1-C4): track 106.1 -> 136.5 mm
- net Net-(U1-C8): track 167.0 -> 196.1 mm, vias 4 -> 6
- net Net-(U1-C9): track 122.1 -> 149.8 mm
- net Net-(MCP1-GPA5): track 0.00 -> 26.6 mm
- net Net-(U1-C2): track 102.2 -> 125.2 mm
- net Net-(U1-C3): track 98.8 -> 121.6 mm
- net Net-(U1-R1): track 146.6 -> 167.1 mm
- net Net-(U1-C1): track 103.4 -> 116.9 mm
- net Net-(U1-R4): track 257.5 -> 270.2 mm
- net Net-(U1-R2): track 172.7 -> 182.5 mm
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