File: hardware/kicad-keyboard/keyboard/keyboard.kicad_sch (KiCad schematic)
At the start: 89 parts, among them SW1 SW_Push, SW10 SW_Push, SW11 SW_Push, SW12 SW_Push, SW13 SW_Push, SW14 SW_Push, SW15 SW_Push, SW16 SW_Push, SW17 SW_Push, SW18 SW_Push, SW19 SW_Push, SW2 SW_Push, SW20 SW_Push, SW21 SW_Push, SW22 SW_Push, SW23 SW_Push, SW24 SW_Push, SW25 SW_Push, SW26 SW_Push, SW27 SW_Push, SW28 SW_Push, SW29 SW_Push, SW3 SW_Push, SW30 SW_Push, SW31 SW_Push, SW32 SW_Push, SW33 SW_Push, SW34 SW_Push, SW35 SW_Push, SW36 SW_Push, SW37 SW_Push, SW38 SW_Push, SW39 SW_Slide_DPDT, SW4 SW_Push, SW5 SW_Push, SW6 SW_Push, SW7 SW_Push, SW8 SW_Push, SW9 SW_Push

Commit message: Keyboard pcb fix (#74)
* fix: Fixes push button switch footprint pad assignation

* fix: Fixes rotary encoder footprint pad assignation

* fix: Reannotates schematic components

* fix: Reworks keyboard PCB

* chore: KiCad updates

* chore: keyboard PCB review done

* fix: Numerotation fix

* chore: Adds some 3D models
Parts:
- D12: renamed from U3; footprint (none) -> Lilyspad:led
- renumbered D30 to D11, D11 to D13, D12 to D14, D13 to D15, D14 to D16, D15 to D17, D16 to D18, D17 to D19, D18 to D20, D19 to D21, D20 to D22, D38 to D23, D21 to D24, D22 to D25, D23 to D26, D24 to D27, D25 to D28, D26 to D29, D27 to D30, D29 to D31, D28 to D32, D31 to D33, D32 to D34, D33 to D35, D34 to D36, D35 to D37, D36 to D38, D37 to D39, M4 to M3, M3 to M4, MCP23017 to MCP1, R4 to R1, R1 to R2, R2 to R3, R3 to R4, SW39 to SW1, SW9 to SW10, SW10 to SW11, SW30 to SW12, SW11 to SW13, SW12 to SW14, SW13 to SW15, SW14 to SW16, SW15 to SW17, SW16 to SW18, SW17 to SW19, SW1 to SW2, SW18 to SW20, SW19 to SW21, SW20 to SW22, SW38 to SW23, SW40 to SW24, SW21 to SW25, SW22 to SW26, SW23 to SW27, SW24 to SW28, SW25 to SW29, SW2 to SW3, SW26 to SW30, SW27 to SW31, SW28 to SW32, SW29 to SW33, SW31 to SW34, SW32 to SW35, SW33 to SW36, SW34 to SW37, SW35 to SW38, SW36 to SW39, SW3 to SW4, SW37 to SW40, SW4 to SW5, SW5 to SW6, SW6 to SW7, SW7 to SW8, SW8 to SW9
