File: hardware/pcbs/main_pcb/main_pcb.kicad_sch (KiCad schematic)
At the start: 17 parts, among them J5 Conn_01x06, SW1 SW_Push, U5 ATmega2560-16A

Commit message: feat(main PCB): Reworks schematic
Parts:
- C11, C14: symbol Device:C -> Lilybrary:Capacitor
- D1, D2, D3, D5: symbol Device:LED -> Lilybrary:LED
- J5: symbol Connector_Generic:Conn_01x06 -> Lilybrary:Conn_01x06
- R2, R3, R4, R5, R7: symbol Device:R -> Lilybrary:Resistor
- SW1: symbol Switch:SW_Push -> Lilybrary:SW_Push
- TP6, TP7: symbol Connector:TestPoint -> Lilybrary:TestPoint
- U5: footprint Package_QFP:TQFP-100_14x14mm_P0.5mm -> Lilibrary:ATmega2560-16AU; symbol MCU_Microchip_ATmega:ATmega2560-16A -> Lilybrary:ATmega2560-16A
Connections:
- net MISO: now also TP7. (1); no longer TP7.1
- net MOSI: now also TP6. (1); no longer TP6.1
- net VCC: now also D1.1 (K), D2.1 (K), D3.1 (K), D5.1 (K); no longer D1.2 (A), D2.2 (A), D3.2 (A), D5.2 (A)
- net at R5.2: now also D3.2 (A); no longer D3.1 (K)
- net at R2.2: now also D1.2 (A); no longer D1.1 (K)
- net at R7.2: now also D5.2 (A); no longer D5.1 (K)
- net at R3.2: now also D2.2 (A); no longer D2.1 (K)
Other:
- company: (none) -> Lily's Pad
- title: (none) -> Main PCB
- moved on the sheet: C11, C14, D1, D2, D3, D5, J5, SW1, U5, U7

Commit message: feat(main PCB): Fixes main PCB routing issue
Connections:
- net MISO: now also TP7.1; no longer TP7. (1)
- net MOSI: now also TP6.1; no longer TP6. (1)
Changed lines of the file:
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@@
 			)
 		)
-		(pin ""
+		(pin "1"
 		)
 		(instances
@@
 			)
 		)
-		(pin ""
-		)
-		(instances
+		(pin "1"
+		)
+		(instances
