File: hardware/pcbs/main_pcb/main_pcb.kicad_pcb (KiCad board)
At the start: 2 copper layers, 130 x 100 mm, 62 parts, among them J1 Conn_01x02, J2 Conn_01x07, J3 Conn_01x07, J4 Conn_01x13, J5 Conn_01x06, J6 Conn_01x02, J7 USB_C_Receptacle_USB2.0_14P, SW1 SW_Push, U1 TXB0104D, U2 TXB0104D, U3 TXB0104D, U4 AMS1117-3.3, U5 ATmega2560-16A, U6 CH340C, Y1 Crystal_GND24

Commit message: Maddie/main pcb schematic cleaning (#88)
* feat(main PCB): Reworks schematic

* feat(main PCB): Removes no longer used BL pin 01x02 header

* feat(main PCB): Fixes main PCB routing issue

* chore: Reworks main PCB schematic/PCB

* chore: Removes old csv file
Parts:
- removed J1: Conn_01x02, Lilibrary:JST XH 2 pins
- removed REF** (x4): Mounting_Hole_3.2mm_M3, Lilibrary:Mounting_Hole_3.2mm_M3
- U1, U2, U3: footprint Package_SO:SOIC-14_3.9x8.7mm_P1.27mm -> Lilibrary:SOIC-14_TXB0104DR
- U4: footprint Package_TO_SOT_SMD:SOT-223-3_TabPin2 -> Lilibrary:SOT-223-3_TabPin2_AMS1117
- U5: footprint Package_QFP:TQFP-100_14x14mm_P0.5mm -> Lilibrary:ATmega2560-16AU
- turned D1 to 0 degrees
- turned D2 to 0 degrees
- turned D3 to 0 degrees
- turned D4 to -90 degrees
- turned D5 to 0 degrees
- turned U4 to 0 degrees
Connections:
- D1 pad 1: Net-(D1-K) -> VCC
- D1 pad 2: VCC -> Net-(D1-A)
- D2 pad 1: Net-(D2-K) -> VCC
- D2 pad 2: VCC -> Net-(D2-A)
- D3 pad 1: Net-(D3-K) -> VCC
- D3 pad 2: VCC -> Net-(D3-A)
- D4 pad 1: GND -> Net-(D4-K)
- D4 pad 2: Net-(D4-A) -> GND
- D5 pad 1: Net-(D5-K) -> VCC
- D5 pad 2: VCC -> Net-(D5-A)
- J2 pad 5: /Screens/DC-3V3 -> /Screens/DC_3V3
- J3 pad 5: /Screens/DC-3V3 -> /Screens/DC_3V3
- J4 pad 5: /Screens/DC-3V3 -> /Screens/DC_3V3
- R2 pad 2: Net-(D1-K) -> Net-(D1-A)
- R3 pad 2: Net-(D2-K) -> Net-(D2-A)
- R5 pad 2: Net-(D3-K) -> Net-(D3-A)
- R6 pad 2: Net-(D4-A) -> Net-(D4-K)
- R7 pad 2: Net-(D5-K) -> Net-(D5-A)
- TP3 pad 1: /Screens/DC-3V3 -> /Screens/DC_3V3
- U2 pad 2: /Screens/SCK_3V3 -> /Screens/DC_3V3
- U2 pad 3: /Screens/MISO_3V3 -> /Screens/SCK_3V3
- U2 pad 5: /Screens/DC-3V3 -> /Screens/MISO_3V3
Routing:
- net /Screens/DC_3V3: track 0.00 -> 118.2 mm, vias 0 -> 6
- net /Screens/DC-3V3: track 111.5 -> 0.00 mm, vias 6 -> 0
- net /Screens/MAIN_SCREEN_BL-3V3: track 27.3 -> 13.7 mm, vias 3 -> 2
- net Net-(D2-K): track 4.92 -> 0.00 mm
- net Net-(D2-A): track 0.00 -> 4.92 mm
- net Net-(D1-K): track 4.92 -> 0.00 mm
- net Net-(D1-A): track 0.00 -> 4.92 mm
- net Net-(D5-K): track 4.65 -> 0.00 mm
- net Net-(D5-A): track 0.00 -> 4.65 mm
- net Net-(D3-K): track 4.65 -> 0.00 mm
- net Net-(D3-A): track 0.00 -> 4.65 mm
- net Net-(D4-K): track 0.00 -> 4.25 mm
- net Net-(D4-A): track 4.25 -> 0.00 mm
- net /Screens/MISO_3V3: track 35.0 -> 36.5 mm, vias 4 -> 6
- net /C2: track 44.6 -> 43.8 mm
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